Commit message: franka: dual arm setting for gazebo

File: franka_description/robots/dual_panda_robot.urdf.xacro (robot description, xacro)
@@ -1,5 +1,5 @@
 <?xml version="1.0"?>
 <robot xmlns:xacro="http://www.ros.org/wiki/xacro"
-       name="dual_panda" >
+       name="dual_franka" >
   <!-- panda -->
   <xacro:include filename="$(find franka_description)/robots/panda_arm.xacro" />
@@ -17,7 +17,7 @@
   <link name="dual_arm_base" >
     <visual>
-      <!--origin xyz="0 -0.4 0" rpy="1.5707963267949 0.0 0.0" /-->
-      <geometry>
-        <mesh filename="package://ur_e_description/meshes/ur5e/dual_ur5_base.stl" />
+      <origin xyz="0 -0.4 0" rpy="1.5707963267949 0.0 0.0" />
+      <geometry>
+        <mesh filename="package://franka_description/meshes/dual_franka_base.dae" scale="0.001 0.001 0.001" />
       </geometry>
       <material name="misumi">
@@ -26,14 +26,14 @@
     </visual>
     <collision>
-      <!--origin xyz="0 -0.4 0" rpy="1.5707963267949 0.0 0.0" /-->
-      <geometry>
-        <mesh filename="package://ur_e_description/meshes/ur5e/dual_ur5_base.stl" />
+      <origin xyz="0 -0.4 0" rpy="1.5707963267949 0.0 0.0" />
+      <geometry>
+        <mesh filename="package://franka_description/meshes/dual_franka_base.dae" scale="0.001 0.001 0.001" />
       </geometry>
     </collision>
     <inertial>
       <mass value="1000" />
-      <origin rpy="0 0 0" xyz="0.0 0.0 0.8"/>
-      <inertia ixx="1.0" ixy="0.0" ixz="0.0"
-               iyy="1.0" iyz="0.0" izz="1.0" />
+      <origin rpy="0 0 0" xyz="0.0 0.0 0.2"/>
+      <inertia ixx="10.0" ixy="0.0" ixz="0.0"
+               iyy="10.0" iyz="0.0" izz="10.0" />
     </inertial>
   </link>
@@ -129,5 +129,5 @@
       <origin rpy="1.5707963267949 0.0 0.0" xyz="0 -0.75 0"/>
       <geometry>
-        <mesh filename="package://ur_e_description/meshes/ur5e/dual_ur5_booth.stl"
+        <mesh filename="package://franka_description/meshes/dual_franka_booth.stl"
               scale="0.001 0.001 0.001" />
       </geometry>
@@ -139,5 +139,5 @@
       <origin rpy="1.5707963267949 0.0 0.0" xyz="0 -0.75 0"/>
       <geometry>
-        <mesh filename="package://ur_e_description/meshes/ur5e/dual_ur5_booth.stl"
+        <mesh filename="package://franka_description/meshes/dual_franka_booth.stl"
               scale="0.001 0.001 0.001" />
       </geometry>
@@ -175,10 +175,109 @@
   </joint>
   <!-- pan_tilt -->
-  <xacro:include filename="$(find ur_e_description)/pan_tilt/pan_tilt_kinect.urdf.xacro" />
+  <xacro:include filename="$(find franka_description)/pan_tilt/pan_tilt_kinect.urdf.xacro" />
   <xacro:pan_tilt_kinect />
-  <joint name="" type="fixed" >
+  <joint name="base_to_head" type="fixed" >
     <parent link="dual_arm_base" />
     <child  link="pan_tilt_BASE" />
     <origin rpy="0.0 0.0 -1.5707963267949" xyz="0.08 0.0 1.505"/>
   </joint>
+  <!-- gazebo -->
+  <xacro:macro name="gazebo_transmission" params="joint_name" >
+    <transmission name="${joint_name}_trans">
+      <type>transmission_interface/SimpleTransmission</type>
+      <joint name="${joint_name}">
+        <hardwareInterface>hardware_interface/VelocityJointInterface</hardwareInterface>
+      </joint>
+      <actuator name="${joint_name}_motor">
+        <hardwareInterface>hardware_interface/VelocityJointInterface</hardwareInterface>
+        <mechanicalReduction>1</mechanicalReduction>
+      </actuator>
+    </transmission>
+  </xacro:macro>
+  <xacro:gazebo_transmission joint_name="right_joint1" />
+  <xacro:gazebo_transmission joint_name="right_joint2" />
+  <xacro:gazebo_transmission joint_name="right_joint3" />
+  <xacro:gazebo_transmission joint_name="right_joint4" />
+  <xacro:gazebo_transmission joint_name="right_joint5" />
+  <xacro:gazebo_transmission joint_name="right_joint6" />
+  <xacro:gazebo_transmission joint_name="right_joint7" />
+  <xacro:gazebo_transmission joint_name="left_joint1" />
+  <xacro:gazebo_transmission joint_name="left_joint2" />
+  <xacro:gazebo_transmission joint_name="left_joint3" />
+  <xacro:gazebo_transmission joint_name="left_joint4" />
+  <xacro:gazebo_transmission joint_name="left_joint5" />
+  <xacro:gazebo_transmission joint_name="left_joint6" />
+  <xacro:gazebo_transmission joint_name="left_joint7" />
+  <xacro:gazebo_transmission joint_name="right_finger_joint1" />
+  <xacro:gazebo_transmission joint_name="right_finger_joint2" />
+  <xacro:gazebo_transmission joint_name="left_finger_joint1" />
+  <xacro:gazebo_transmission joint_name="left_finger_joint2" />
+  <!-- create camera frame-->
+  <link name="fisheye_frame" />
+  <joint name="fisheye_fixed_joint" type="fixed">
+    <parent link="dual_arm_base"/>
+    <child link="fisheye_frame"/>
+    <origin xyz="0.07 0 1.9" rpy="0 1.3 0"/>
+  </joint>
+  <!-- camera -->
+  <gazebo reference="fisheye_frame">
+    <sensor name="fisheye_camera_sensor" type="wideanglecamera" >
+      <!--pose>${pose}</pose-->
+      <always_on>true</always_on>
+      <update_rate>15</update_rate>
+      <visualize>false</visualize>
+      <camera name="fisheye_camera">
+        <horizontal_fov>3.14</horizontal_fov>
+        <image>
+          <width>2048</width>
+          <height>2048</height>
+          <format>R8G8B8</format>
+        </image>
+        <clip>
+          <near>0.02</near>
+          <far>300</far>
+        </clip>
+        <lens> <!-- for Fisheye -->
+          <!-- type: gnomonical, stereographic, equidistant, equisolid_angle, orthographic, custom -->
+          <!-- More information here: https://en.wikipedia.org/wiki/Fisheye_lens#Mapping_function -->
+          <!--type>equidistant</type-->
+          <type>custom</type>  <!-- manually defined mapping function r = c1*f*fun(theta/c2 + c3) -->
+          <custom_function>
+            <c1>2</c1>
+            <c2>2</c2>
+            <c3>0</c3>
+            <f>0.63661977</f> <!-- ( 2.0 / pi ) -->
+            <fun>id</fun> <!-- one of sin,tan,id -->
+          </custom_function>
+          <!-- if it is set to `true` your horizontal FOV will ramain as defined -->
+          <!-- othervise it depends on lens type and custom function, if there is one -->
+          <scale_to_hfov>false</scale_to_hfov>
+          <cutoff_angle>1.5707</cutoff_angle> <!-- clip everything that is outside of this angle -->
+          <!-- resolution of the cubemap texture, the highter it is - the sharper is your image -->
+          <env_texture_size>2048</env_texture_size>
+        </lens>
+      </camera>
+      <plugin name="camera_controller" filename="libgazebo_ros_camera.so">
+        <alwaysOn>true</alwaysOn>
+        <updateRate>0.0</updateRate><!-- ? -->
+        <cameraName>fisheye_camera</cameraName>
+        <imageTopicName>image_raw</imageTopicName>
+        <cameraInfoTopicName>camera_info</cameraInfoTopicName>
+        <frameName>fisheye_frame</frameName>
+        <hackBaseline>0.07</hackBaseline>
+        <distortionK1>0.0</distortionK1>
+        <distortionK2>0.0</distortionK2>
+        <distortionK3>0.0</distortionK3>
+        <distortionT1>0.0</distortionT1>
+        <distortionT2>0.0</distortionT2>
+      </plugin>
+    </sensor>
+  </gazebo>
+  <gazebo>
+    <plugin name="gazebo_ros_control" filename="libgazebo_ros_control.so">
+      <!--robotNamespace>/</robotNamespace-->
+      <legacyModeNS>false</legacyModeNS>
+      <robotSimType>gazebo_ros_control/DefaultRobotHWSim</robotSimType>
+    </plugin>
+  </gazebo>
 </robot>

File: franka_description/robots/hand.xacro (robot description, xacro)
@@ -11,4 +11,9 @@
     </xacro:unless>
     <link name="${ns}_hand">
+      <inertial>
+        <mass value="0.01"/>
+        <origin rpy="0 0 0" xyz="0.0 0.0 0.0"/>
+        <inertia ixx="0.000001" ixy="0.0" ixz="0.0" iyy="0.000001" iyz="0.0" izz="0.000001"/>
+      </inertial>
       <visual>
         <geometry>
@@ -16,4 +21,11 @@
         </geometry>
       </visual>
+      <collision>
+        <origin xyz="0.0 0.0 0.0285" />
+        <geometry>
+          <box size="0.056 0.2 0.074" />
+        </geometry>
+      </collision>
+      <!--
       <collision>
         <origin xyz="0 0 0.04" rpy="0 ${pi/2} ${pi/2}"/>
@@ -52,6 +64,12 @@
         </geometry>
       </collision>
+      -->
     </link>
     <link name="${ns}_leftfinger">
+  <inertial>
+     <mass value="0.014505"/>
+     <origin rpy="0 0 0" xyz="3.299713e-07 0.013131 0.027017"/>
+     <inertia ixx="4.338623e-06" ixy="0.0" ixz="0.0" iyy="4.027488e-06" iyz="0.0" izz="1.377502e-06"/>
+  </inertial>
       <visual>
         <geometry>
@@ -59,6 +77,17 @@
         </geometry>
       </visual>
+      <collision>
+        <origin xyz="0.0 0.0131 0.027" />
+        <geometry>
+          <box size="0.021 0.02643 0.0538" />
+        </geometry>
+      </collision>
     </link>
     <link name="${ns}_rightfinger">
+  <inertial>
+     <mass value="0.014505"/>
+     <origin rpy="0 0 0" xyz="3.299713e-07 0.013131 0.027017"/>
+     <inertia ixx="4.338623e-06" ixy="0.0" ixz="0.0" iyy="4.027488e-06" iyz="0.0" izz="1.377502e-06"/>
+  </inertial>
       <visual>
         <origin xyz="0 0 0" rpy="0 0 ${pi}"/>
@@ -67,4 +96,10 @@
         </geometry>
       </visual>
+      <collision>
+        <origin xyz="0.0 -0.0131 0.027" rpy="0 0 ${pi}"/>
+        <geometry>
+          <box size="0.021 0.02643 0.0538" />
+        </geometry>
+      </collision>
    </link>
     <joint name="${ns}_finger_joint1" type="prismatic">

File: franka_description/robots/panda_arm.xacro (robot description, xacro)
@@ -12,4 +12,9 @@
     </xacro:unless>
     <link name="${arm_id}_link0">
+  <inertial>
+     <mass value="2.90428"/>
+     <origin rpy="0 0 0" xyz="-0.041271 -1.158905e-05 0.07"/>
+     <inertia ixx="0.013404" ixy="0.0" ixz="0.0" iyy="0.017065" iyz="0.0" izz="0.020982"/>
+  </inertial>
       <visual>
         <geometry>
@@ -37,4 +42,9 @@
     </link>
     <link name="${arm_id}_link1">
+  <inertial>
+     <mass value="2.43555"/>
+     <origin rpy="0 0 0" xyz="-6.740570e-06 -0.037189 -0.068499"/>
+     <inertia ixx="0.019285" ixy="0.0" ixz="0.0" iyy="0.014839" iyz="0.0" izz="0.009358"/>
+  </inertial>
       <visual>
         <geometry>
@@ -70,4 +80,9 @@
     </joint>
     <link name="${arm_id}_link2">
+  <inertial>
+     <mass value="2.45569"/>
+     <origin rpy="0 0 0" xyz="-1.344109e-05 -0.069488 0.037195"/>
+     <inertia ixx="0.019648" ixy="0.0" ixz="0.0" iyy="0.009436" iyz="0.0" izz="0.015168"/>
+  </inertial>
       <visual>
         <geometry>
@@ -103,4 +118,9 @@
     </joint>
     <link name="${arm_id}_link3">
+  <inertial>
+     <mass value="2.73471"/>
+     <origin rpy="0 0 0" xyz="0.041242 0.028026 -0.032999"/>
+     <inertia ixx="0.013344" ixy="0.0" ixz="0.0" iyy="0.015505" iyz="0.0" izz="0.01473"/>
+  </inertial>
       <visual>
         <geometry>
@@ -136,4 +156,9 @@
     </joint>
     <link name="${arm_id}_link4">
+  <inertial>
+     <mass value="2.78106"/>
+     <origin rpy="0 0 0" xyz="-0.041256 0.0345 0.028032"/>
+     <inertia ixx="0.013816" ixy="0.0" ixz="0.0" iyy="0.014979" iyz="0.0" izz="0.016014"/>
+  </inertial>
       <visual>
         <geometry>
@@ -169,4 +194,9 @@
     </joint>
     <link name="${arm_id}_link5">
+  <inertial>
+     <mass value="3.07672"/>
+     <origin rpy="0 0 0" xyz="-8.943558e-06 0.03747 -0.103401"/>
+     <inertia ixx="0.033599" ixy="0.0" ixz="0.0" iyy="0.027932" iyz="0.0" izz="0.011871"/>
+  </inertial>
       <visual>
         <geometry>
@@ -220,4 +250,9 @@
     </joint>
     <link name="${arm_id}_link6">
+  <inertial>
+     <mass value="1.16471"/>
+     <origin rpy="0 0 0" xyz="0.042059 0.015232 0.006132"/>
+     <inertia ixx="0.002689" ixy="0.0" ixz="0.0" iyy="0.004117" iyz="0.0" izz="0.004855"/>
+  </inertial>
       <visual>
         <geometry>
@@ -253,4 +288,9 @@
     </joint>
     <link name="${arm_id}_link7">
+  <inertial>
+     <mass value="0.418267"/>
+     <origin rpy="0 0 0" xyz="0.01864 0.018625 0.0794"/>
+     <inertia ixx="0.000652" ixy="0.0" ixz="0.0" iyy="0.000652" iyz="0.0" izz="0.001095"/>
+  </inertial>
       <visual>
         <geometry>
@@ -286,4 +326,9 @@
     </joint>
     <link name="${arm_id}_link8">
+      <inertial>
+        <mass value="0.01"/>
+        <origin rpy="0 0 0" xyz="0.0 0.0 0.0"/>
+        <inertia ixx="0.000001" ixy="0.0" ixz="0.0" iyy="0.000001" iyz="0.0" izz="0.000001"/>
+      </inertial>
       <collision>
         <origin xyz="0.0424 0.0424 -0.0250" rpy="${pi} ${pi/2} ${pi/2}"/>

Commit message: update

File: franka_description/robots/dual_panda_robot.urdf.xacro (robot description, xacro)
@@ -9,8 +9,8 @@
   <xacro:arg name="arm_id_2" default="left" />
   <!-- right arm with gripper -->
-  <xacro:panda_arm arm_id="$(arg arm_id_1)" connected_to="fixed_base"  xyz="0 -0.3 0" safety_distance="0.03"/>
+  <xacro:panda_arm arm_id="$(arg arm_id_1)" connected_to="fixed_base"  xyz="-0.02 -0.3 0.0" safety_distance="0.03"/>
   <xacro:hand ns="$(arg arm_id_1)" rpy="0 0 ${-pi/4}" connected_to="$(arg arm_id_1)_link8" safety_distance="0.03"/>
   <!-- left arm with gripper -->
-  <xacro:panda_arm arm_id="$(arg arm_id_2)" connected_to="fixed_base"  xyz="0 0.3 0" safety_distance="0.03"/>
+  <xacro:panda_arm arm_id="$(arg arm_id_2)" connected_to="fixed_base"  xyz="-0.02  0.3 0.0" safety_distance="0.03"/>
   <xacro:hand ns="$(arg arm_id_2)" rpy="0 0 ${-pi/4}" connected_to="$(arg arm_id_2)_link8" safety_distance="0.03"/>
   <link name="fixed_base" />
@@ -43,5 +43,5 @@
     <origin xyz="-0.08 0.0 0.8" rpy="0.0 0.0 0.0" />
   </joint>
-  <link name="table_plane">
+  <!--link name="table_plane">
     <visual>
       <origin xyz="0.3 0 0.01" />
@@ -59,5 +59,5 @@
       </geometry>
     </collision>
-  </link>
+  </link-->
   <link name="controller_plane0">
     <visual>
@@ -80,9 +80,9 @@
     </visual>
   </link>
-  <joint name="base_to_table_plane" type="fixed">
+  <!--joint name="base_to_table_plane" type="fixed">
     <parent link="dual_arm_base" />
     <child  link="table_plane" />
     <origin xyz="0.0 0.0 0.8" rpy="0.0 0.0 0.0" />
-  </joint>
+  </joint-->
   <joint name="base_to_c_plane0" type="fixed">
     <parent link="dual_arm_base" />
@@ -157,5 +157,6 @@
    <visual>
      <geometry>
-       <box size="0.03 0.817 0.342"/>
+       <!--box size="0.03 0.817 0.342"/--> <!-- 34inch wide -->
+       <box size="0.015 0.165 0.150"/> <!-- 12inch -->
      </geometry>
      <material name="Display">
@@ -165,5 +166,6 @@
    <collision>
      <geometry>
-       <box size="0.03 0.817 0.342"/>
+       <!--box size="0.03 0.817 0.342"/-->
+       <box size="0.015 0.165 0.150"/> <!-- 12inch -->
      </geometry>
    </collision>
@@ -172,5 +174,5 @@
     <parent link="dual_arm_base"/>
     <child  link="display"/>
-    <origin rpy="0.0 0.2 0.0" xyz="0.0 0.0 1.72"/>
+    <origin rpy="0.0 0.2 0.0" xyz="0.0 0.0 1.66"/>
   </joint>
   <!-- pan_tilt -->
