Commit message: add fixed connection to world

File: franka_description/dual_franka.urdf (robot description, URDF)
Before this commit: robot dual_franka, 41 links, 40 joints
Links:
- added link world
Joints:
- added joint fix_to_world: type fixed, parent world, child dual_arm_base

Commit message: modify model path of pan-tilt from ur_e_description to franka_description, also re-generate dual_franka.l

File: franka_description/dual_franka.urdf (robot description, URDF)
Before this commit: robot dual_franka, 42 links, 41 joints
Links:
- removed link world
- link camera_link: geometry collision box size=0.07271 0.27794 0.073; visual mesh filename=package://franka_description/pan_tilt/meshes/kinect.dae
- link pan_tilt_BASE: geometry collision mesh filename=package://franka_description/pan_tilt/meshes/fr12_x102.dae scale=1.000000 1.000000 1.000000; collision mesh filename=package://franka_description/pan_tilt/meshes/xm430_dynamixe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 scale=1.000000 1.000000 1.000000
- link pan_tilt_LINK0: geometry collision mesh filename=package://franka_description/pan_tilt/meshes/fr12_h101s.dae scale=1.000000 1.000000 1.000000; visual mesh filename=package://franka_description/pan_tilt/meshes/fr12_h101s.dae scale=1.000000 1.000000 1.000000
- link pan_tilt_LINK1: geometry collision mesh filename=package://franka_description/pan_tilt/meshes/fr12_h101.dae scale=1.000000 1.000000 1.000000; visual mesh filename=package://franka_description/pan_tilt/meshes/fr12_h101.dae scale=1.000000 1.000000 1.000000
- link pan_tilt_PAN_BASE: geometry collision mesh filename=package://franka_description/pan_tilt/meshes/xm430_dynamixe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 scale=1.000000 1.000000 1.000000; visual mesh filename=package://franka_description/pan_tilt/meshes/xm430_dynamixe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 scale=1.000000 1.000000 1.000000
Joints:
- removed joint fix_to_world

File: franka_description/pan_tilt/kinect.urdf.xacro (robot description, xacro)
@@ -2,5 +2,5 @@
 <!-- copy from openni_description -->
 <robot name="sensor_openni" xmlns:xacro="http://ros.org/wiki/xacro">
-  <xacro:include filename="$(find ur_e_description)/pan_tilt/kinect_gazebo.urdf.xacro" />
+  <xacro:include filename="$(find franka_description)/pan_tilt/kinect_gazebo.urdf.xacro" />
   <!-- Parameterised in part by the values in turtlebot_properties.urdf.xacro -->
   <xacro:macro name="sensor_kinect" params="parent cam_px cam_py cam_pz cam_or cam_op cam_oy">
@@ -26,5 +26,5 @@
        <origin xyz="0 0 0" rpy="0 0 ${M_PI/2}"/>
         <geometry>
-         <mesh filename="package://ur_e_description/pan_tilt/meshes/kinect.dae"/>
+         <mesh filename="package://franka_description/pan_tilt/meshes/kinect.dae"/>
         </geometry>
       </visual>

File: franka_description/pan_tilt/pan_tilt_base.urdf.xacro (robot description, xacro)
@@ -38,5 +38,5 @@
         <origin xyz="0.000000 0.000000 0.000000" rpy="0.00000000 -0.00000000 0.00000000"/>
         <geometry>
-          <mesh filename="package://ur_e_description/pan_tilt/meshes/xm430_dynamixel.dae" scale="1.000000 1.000000 1.000000"/>
+          <mesh filename="package://franka_description/pan_tilt/meshes/xm430_dynamixel.dae" scale="1.000000 1.000000 1.000000"/>
         </geometry>
       </visual>
@@ -44,5 +44,5 @@
         <origin xyz="0.000000 0.000000 0.000000" rpy="0.00000000 -0.00000000 0.00000000"/>
         <geometry>
-          <mesh filename="package://ur_e_description/pan_tilt/meshes/xm430_dynamixel.dae" scale="1.000000 1.000000 1.000000"/>
+          <mesh filename="package://franka_description/pan_tilt/meshes/xm430_dynamixel.dae" scale="1.000000 1.000000 1.000000"/>
         </geometry>
       </collision>
@@ -50,5 +50,5 @@
         <origin xyz="-0.000000 -0.000000 -0.003000" rpy="-1.57079633 0.00000000 3.14159265"/>
         <geometry>
-          <mesh filename="package://ur_e_description/pan_tilt/meshes/fr12_x102.dae" scale="1.000000 1.000000 1.000000"/>
+          <mesh filename="package://franka_description/pan_tilt/meshes/fr12_x102.dae" scale="1.000000 1.000000 1.000000"/>
         </geometry>
       </visual>
@@ -56,5 +56,5 @@
         <origin xyz="-0.000000 -0.000000 -0.003000" rpy="-1.57079633 0.00000000 3.14159265"/>
         <geometry>
-          <mesh filename="package://ur_e_description/pan_tilt/meshes/fr12_x102.dae" scale="1.000000 1.000000 1.000000"/>
+          <mesh filename="package://franka_description/pan_tilt/meshes/fr12_x102.dae" scale="1.000000 1.000000 1.000000"/>
         </geometry>
       </collision>
@@ -70,5 +70,5 @@
         <origin xyz="0.000000 0.000000 -0.019000" rpy="0.00000000 1.57079633 0.00000000"/>
         <geometry>
-          <mesh filename="package://ur_e_description/pan_tilt/meshes/fr12_h101s.dae" scale="1.000000 1.000000 1.000000"/>
+          <mesh filename="package://franka_description/pan_tilt/meshes/fr12_h101s.dae" scale="1.000000 1.000000 1.000000"/>
         </geometry>
       </visual>
@@ -76,5 +76,5 @@
         <origin xyz="0.000000 0.000000 -0.019000" rpy="0.00000000 1.57079633 0.00000000"/>
         <geometry>
-          <mesh filename="package://ur_e_description/pan_tilt/meshes/fr12_h101s.dae" scale="1.000000 1.000000 1.000000"/>
+          <mesh filename="package://franka_description/pan_tilt/meshes/fr12_h101s.dae" scale="1.000000 1.000000 1.000000"/>
         </geometry>
       </collision>
@@ -98,5 +98,5 @@
         <origin xyz="0.000000 0.000000 0.000000" rpy="0.00000000 -0.00000000 0.00000000"/>
         <geometry>
-          <mesh filename="package://ur_e_description/pan_tilt/meshes/xm430_dynamixel.dae" scale="1.000000 1.000000 1.000000"/>
+          <mesh filename="package://franka_description/pan_tilt/meshes/xm430_dynamixel.dae" scale="1.000000 1.000000 1.000000"/>
         </geometry>
       </visual>
@@ -104,5 +104,5 @@
         <origin xyz="0.000000 0.000000 0.000000" rpy="0.00000000 -0.00000000 0.00000000"/>
         <geometry>
-          <mesh filename="package://ur_e_description/pan_tilt/meshes/xm430_dynamixel.dae" scale="1.000000 1.000000 1.000000"/>
+          <mesh filename="package://franka_description/pan_tilt/meshes/xm430_dynamixel.dae" scale="1.000000 1.000000 1.000000"/>
         </geometry>
       </collision>
@@ -118,5 +118,5 @@
         <origin xyz="0.000000 0.000000 -0.019000" rpy="0.00000000 1.57079633 1.57079633"/>
         <geometry>
-          <mesh filename="package://ur_e_description/pan_tilt/meshes/fr12_h101.dae" scale="1.000000 1.000000 1.000000"/>
+          <mesh filename="package://franka_description/pan_tilt/meshes/fr12_h101.dae" scale="1.000000 1.000000 1.000000"/>
         </geometry>
       </visual>
@@ -124,5 +124,5 @@
         <origin xyz="0.000000 0.000000 -0.019000" rpy="0.00000000 1.57079633 1.57079633"/>
         <geometry>
-          <mesh filename="package://ur_e_description/pan_tilt/meshes/fr12_h101.dae" scale="1.000000 1.000000 1.000000"/>
+          <mesh filename="package://franka_description/pan_tilt/meshes/fr12_h101.dae" scale="1.000000 1.000000 1.000000"/>
         </geometry>
       </collision>

File: franka_description/pan_tilt/pan_tilt_kinect.urdf.xacro (robot description, xacro)
@@ -1,6 +1,6 @@
 <?xml version="1.0" ?>
 <robot xmlns:xacro="http://ros.org/wiki/xacro">
-  <xacro:include filename="$(find ur_e_description)/pan_tilt/pan_tilt_base.urdf.xacro" />
-  <xacro:include filename="$(find ur_e_description)/pan_tilt/kinect.urdf.xacro" />
+  <xacro:include filename="$(find franka_description)/pan_tilt/pan_tilt_base.urdf.xacro" />
+  <xacro:include filename="$(find franka_description)/pan_tilt/kinect.urdf.xacro" />
   <!--xacro:include filename="$(find openni_description)/model/kinect.urdf.xacro" /-->
   <xacro:macro name="pan_tilt_kinect"

File: franka_description/pan_tilt/pan_tilt_kinect_robot.urdf.xacro (robot description, xacro)
@@ -2,5 +2,5 @@
 <robot name="pan_tilt_kinect_robot"
        xmlns:xacro="http://www.ros.org/wiki/xacro">
-  <xacro:include filename="$(find ur_e_description)/pan_tilt/pan_tilt_kinect.urdf.xacro" />
+  <xacro:include filename="$(find franka_description)/pan_tilt/pan_tilt_kinect.urdf.xacro" />
   <xacro:pan_tilt_kinect />
 </robot>
